Commit message: fix

File: src/yixuan_utilities/assets/robot/vega-urdf/vega_no_effector.urdf (robot description, URDF)
Before this commit: robot vega-1, 45 links, 44 joints
Joints:
- joint torso_j3: limit lower=-1.570 upper=0.0 effort=380 velocity=0.9 -> lower=-1.570 upper=1.570 effort=380 velocity=0.9
